Commit message: Switched to a better simulator fork and removed hector_quadrotor package (no longer needed).

File: tum_simulator/cvg_sim_gazebo/urdf/quadrotor.urdf.xacro (robot description, xacro)
@@ -6,5 +6,5 @@
     xmlns:xacro="http://playerstage.sourceforge.net/gazebo/xmlschema/#interface">
     <!-- Included URDF Files -->
-    <include filename="$(find cvg_sim_gazebo)/urdf/quadrotor_base.urdf.xacro" />
+    <xacro:include filename="$(find cvg_sim_gazebo)/urdf/quadrotor_base.urdf.xacro" />
     <!-- Instantiate quadrotor_base_macro once (has no parameters atm) -->
     <quadrotor_base_macro />

File: tum_simulator/cvg_sim_gazebo/urdf/quadrotor_base.urdf.xacro (robot description, xacro)
@@ -5,5 +5,5 @@
 xmlns:xacro="http://ros.org/wiki/xacro"
 >
-  <include filename="$(find cvg_sim_gazebo_plugins)/urdf/quadrotor_plugins.urdf.xacro" />
+  <xacro:include filename="$(find cvg_sim_gazebo_plugins)/urdf/quadrotor_plugins.urdf.xacro" />
   <property name="pi" value="3.1415926535897931" />
   <!-- Main quadrotor link -->

File: tum_simulator/cvg_sim_gazebo/urdf/quadrotor_sensors.urdf.xacro (robot description, xacro)
@@ -7,14 +7,14 @@
     <property name="M_PI" value="3.1415926535897931" />
     <!-- Included URDF Files -->
-    <include filename="$(find cvg_sim_gazebo)/urdf/quadrotor_base.urdf.xacro" />
+    <xacro:include filename="$(find cvg_sim_gazebo)/urdf/quadrotor_base.urdf.xacro" />
     <!-- Instantiate quadrotor_base_macro once (has no parameters atm) -->
     <quadrotor_base_macro />
     <!-- Sonar height sensor -->
-    <include filename="$(find cvg_sim_gazebo)/urdf/sensors/sonar_sensor.urdf.xacro" />
+    <xacro:include filename="$(find cvg_sim_gazebo)/urdf/sensors/sonar_sensor.urdf.xacro" />
     <xacro:sonar_sensor name="sonar" parent="base_link" ros_topic="sonar_height" update_rate="10" min_range="0.01" max_range="3.0" field_of_view="${40*M_PI/180}" ray_count="3">
       <origin xyz="-0.15 0.0 0.0" rpy="0 ${90*M_PI/180} 0"/>
     </xacro:sonar_sensor>
     <!-- Hokuyo UTM-30LX mounted upside down below the quadrotor body
-    <include filename="$(find cvg_sim_gazebo)/urdf/sensors/hokuyo_utm30lx.urdf.xacro" />
+    <xacro:include filename="$(find cvg_sim_gazebo)/urdf/sensors/hokuyo_utm30lx.urdf.xacro" />
     <xacro:hokuyo_utm30lx name="laser0" parent="base_link" ros_topic="scan" update_rate="40" ray_count="1081" min_angle="135" max_angle="-135">
       <origin xyz="0.0 0.0 0.08" rpy="${M_PI} 0 0"/>
@@ -22,10 +22,10 @@
     <!-- The following two cameras should be united to one! -->
     <!-- Forward facing camera -->
-    <include filename="$(find cvg_sim_gazebo)/urdf/sensors/generic_camera.urdf.xacro" />
+    <xacro:include filename="$(find cvg_sim_gazebo)/urdf/sensors/generic_camera.urdf.xacro" />
     <xacro:generic_camera name="front" sim_name="ardrone" parent="base_link" update_rate="60" res_x="640" res_y="360" image_format="R8G8B8" hfov="${81*M_PI/180}">
       <origin xyz="0.21 0.0 0.01" rpy="0 0 0"/>
     </xacro:generic_camera>
     <!-- Downward facing camera -->
-    <include filename="$(find cvg_sim_gazebo)/urdf/sensors/generic_camera.urdf.xacro" />
+    <xacro:include filename="$(find cvg_sim_gazebo)/urdf/sensors/generic_camera.urdf.xacro" />
     <xacro:generic_camera name="bottom" sim_name="ardrone" parent="base_link" update_rate="60" res_x="640" res_y="360" image_format="R8G8B8" hfov="${81*M_PI/180}">
       <origin xyz="0.15 0.0 0.0" rpy="0 -${M_PI/2} 0"/>

File: tum_simulator/cvg_sim_gazebo/urdf/sensors/generic_camera.urdf.xacro (robot description, xacro)
@@ -85,5 +85,5 @@
       </sensor>
       <turnGravityOff>true</turnGravityOff>
-      <material>PR2/Blue</material>
+      <material>Gazebo/Blue</material>
     </gazebo>
     </xacro:macro>

File: tum_simulator/cvg_sim_gazebo_plugins/urdf/quadrotor_sensors.urdf.xacro (robot description, xacro)
@@ -12,5 +12,5 @@
       <plugin name="quadrotor_imu_sim" filename="libhector_gazebo_ros_imu.so">
         <alwaysOn>true</alwaysOn>
-        <updateRate>100.0</updateRate>
+        <updateRate>50.0</updateRate>
         <bodyName>base_link</bodyName>
         <frameId>ardrone_base_link</frameId>
@@ -27,5 +27,5 @@
       <plugin name="quadrotor_baro_sim" filename="libhector_gazebo_ros_baro.so">
         <alwaysOn>true</alwaysOn>
-        <updateRate>10.0</updateRate>
+        <updateRate>50.0</updateRate>
         <bodyName>base_link</bodyName>
         <topicName>pressure_height</topicName>
@@ -37,5 +37,5 @@
       <plugin name="quadrotor_magnetic_sim" filename="libhector_gazebo_ros_magnetic.so">
         <alwaysOn>true</alwaysOn>
-        <updateRate>10.0</updateRate>
+        <updateRate>50.0</updateRate>
         <bodyName>base_link</bodyName>
         <topicName>magnetic</topicName>
@@ -46,12 +46,16 @@
       <plugin name="quadrotor_gps_sim" filename="libhector_gazebo_ros_gps.so">
         <alwaysOn>true</alwaysOn>
-        <updateRate>4.0</updateRate>
+        <updateRate>1.0</updateRate>
         <bodyName>base_link</bodyName>
+        <frameId>gps_base_link</frameId>
         <topicName>fix</topicName>
         <velocityTopicName>fix_velocity</velocityTopicName>
+        <referenceLatitude>37.360500</referenceLatitude>
+        <referenceLongitude>-121.867514</referenceLongitude>
+        <referenceAltitude>136</referenceAltitude>
         <drift>5.0 5.0 5.0</drift>
         <gaussianNoise>0.1 0.1 0.1</gaussianNoise>
         <velocityDrift>0 0 0</velocityDrift>
-        <velocityGaussianNoise>0.1 0.1 0.1</velocityGaussianNoise>
+        <velocityGaussianNoise>0.0 0.0 0.0</velocityGaussianNoise>
       </plugin>
       <plugin name="quadrotor_groundtruth_sim" filename="libgazebo_ros_p3d.so">
