Commit message: added sensor to quadcopter and updated control algorithm

File: simulated_drone/urdf/quadrotor_three_sensors.urdf.xacro (robot description, xacro)
@@ -6,4 +6,5 @@
 xmlns:xacro="http://playerstage.sourceforge.net/gazebo/xmlschema/#interface">
     <property name="M_PI" value="3.1415926535897931" />
+    <property name="FRONT_SENSOR_ANGLE" value="90" />
     <!-- Included URDF Files -->
     <include filename="$(find cvg_sim_gazebo)/urdf/quadrotor_base.urdf.xacro" />
@@ -17,9 +18,13 @@
     <!-- Ultrasonic range sensors -->
     <include filename="$(find cvg_sim_gazebo)/urdf/sensors/sonar_sensor.urdf.xacro" />
-    <xacro:sonar_sensor name="r_front" parent="base_link" ros_topic="range_front" update_rate="10" min_range="0.01" max_range="3.0" field_of_view="${40*M_PI/180}" ray_count="3">
-      <origin xyz="0.21 0.0 0.027" rpy="0 0 0"/>
+    <xacro:sonar_sensor name="r_front_left" parent="base_link" ros_topic="range_front_left" update_rate="10" min_range="0.2" max_range="1.5" field_of_view="${40*M_PI/180}" ray_count="3">
+      <origin xyz="0.21 0.24 0.027" rpy="0 0 ${FRONT_SENSOR_ANGLE/2*M_PI/180}"/>
     </xacro:sonar_sensor>
     <include filename="$(find cvg_sim_gazebo)/urdf/sensors/sonar_sensor.urdf.xacro" />
-    <xacro:sonar_sensor name="r_side" parent="base_link" ros_topic="range_side" update_rate="10" min_range="0.01" max_range="3.0" field_of_view="${40*M_PI/180}" ray_count="3">
+    <xacro:sonar_sensor name="r_front_right" parent="base_link" ros_topic="range_front_right" update_rate="10" min_range="0.2" max_range="1.5" field_of_view="${40*M_PI/180}" ray_count="3">
+      <origin xyz="0.21 -0.24 0.027" rpy="0 0 ${-1*FRONT_SENSOR_ANGLE/2*M_PI/180}"/>
+    </xacro:sonar_sensor>
+    <include filename="$(find cvg_sim_gazebo)/urdf/sensors/sonar_sensor.urdf.xacro" />
+    <xacro:sonar_sensor name="r_side" parent="base_link" ros_topic="range_side" update_rate="10" min_range="0.2" max_range="1.5" field_of_view="${40*M_PI/180}" ray_count="3">
       <origin xyz="0.0 0.24 0.027" rpy="0 0 ${90*M_PI/180}"/>
     </xacro:sonar_sensor>

Commit message: changes for moving sensor to front except for control logic

File: simulated_drone/urdf/quadrotor_three_sensors.urdf.xacro (robot description, xacro)
@@ -26,6 +26,6 @@
     </xacro:sonar_sensor>
     <include filename="$(find cvg_sim_gazebo)/urdf/sensors/sonar_sensor.urdf.xacro" />
-    <xacro:sonar_sensor name="r_side" parent="base_link" ros_topic="range_side" update_rate="10" min_range="0.2" max_range="1.5" field_of_view="${40*M_PI/180}" ray_count="3">
-      <origin xyz="0.0 0.24 0.027" rpy="0 0 ${90*M_PI/180}"/>
+    <xacro:sonar_sensor name="r_front" parent="base_link" ros_topic="range_front" update_rate="10" min_range="0.2" max_range="1.5" field_of_view="${40*M_PI/180}" ray_count="3">
+      <origin xyz="0.21 0.0 0.027" rpy="0 0 ${0*M_PI/180}"/>
     </xacro:sonar_sensor>
     <!-- Hokuyo UTM-30LX mounted upside down below the quadrotor body
